File: KiCad_Files/etuvalo_v2.kicad_pcb (KiCad board)
At the start: 2 copper layers, 59.2 x 57 mm, 38 parts, among them J1 Conn_01x06, J10 Conn_01x01, J11 Conn_01x01, J2 Conn_01x02, J3 Conn_01x02, J4 Conn_01x03, J5 Conn_01x03, J6 Conn_01x03, J7 Conn_01x01, J8 Conn_01x01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

Commit message: Changes
Connections:
- net Exc_sft_reg renamed Sft_reg_clk
- J6 pad 2: PB2 -> Sft_reg_data
- J8 pad 1: PB2 -> Sft_reg_data
- R15 pad 1: PB2 -> Sft_reg_data
- U1 pad 7: PB2 -> Sft_reg_data
Routing:
- net Sft_reg_data: track 0.00 -> 11.3 mm
- net PB2: track 16.2 -> 5.18 mm
Changed lines of the file:
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@@
 	(net 8 "Sw1")
 	(net 9 "UPDI")
-	(net 10 "Exc_sft_reg")
+	(net 10 "Sft_reg_clk")
 	(net 11 "Net-(U1-PB0)")
 	(net 12 "Frontlight_PWM")
@@
 	(net 23 "Thermistor out")
 	(net 24 "Net-(D1-A)")
+	(net 25 "Sft_reg_data")
 	(footprint "Connector_PinSocket_1.27mm:PinSocket_1x01_P1.27mm_Vertical"
 		(layer "F.Cu")
@@
 			(layers "F.Cu" "F.Mask" "F.Paste")
 			(roundrect_rratio 0.25)
-			(net 10 "Exc_sft_reg")
+			(net 10 "Sft_reg_clk")
 			(pinfunction "PB3")
 			(pintype "bidirectional")
@@
 			(layers "F.Cu" "F.Mask" "F.Paste")
 			(roundrect_rratio 0.25)
-			(net 22 "PB2")
+			(net 25 "Sft_reg_data")
 			(pinfunction "PB2")
 			(pintype "bidirectional")
@@
 			(layers "F.Cu" "F.Mask" "F.Paste")
 			(roundrect_rratio 0.192308)
-			(net 22 "PB2")
+			(net 25 "Sft_reg_data")
 			(pintype "passive")
 		)
@@
 			(layers "*.Cu" "*.Mask")
 			(remove_unused_layers no)
-			(net 22 "PB2")
+			(net 25 "Sft_reg_data")
 			(pinfunction "Pin_1")
 			(pintype "passive")
@@
 			(layers "*.Cu" "*.Mask")
 			(remove_unused_layers no)
-			(net 22 "PB2")
+			(net 25 "Sft_reg_data")
 			(pinfunction "Pin_2")
 			(pintype "passive")
@@
 			(layers "*.Cu" "*.Mask")
 			(remove_unused_layers no)
-			(net 10 "Exc_sft_reg")
+			(net 10 "Sft_reg_clk")
 			(pinfunction "Pin_2")
 			(pintype "passive")
@@
 	)
 	(segment
-		(start 144.25 117.4)
-		(end 144.25 117.25)
-		(width 0.5)
-		(layer "F.Cu")
-		(net 22)
-	)
-	(segment
-		(start 144.25 117.25)
-		(end 144.2 117.2)
-		(width 0.5)
-		(layer "F.Cu")
-		(net 22)
-	)
-	(segment
 		(start 140.9 90.7)
 		(end 140.9 89.1)
@@
 	)
 	(segment
-		(start 144.2 117.2)
-		(end 141.3 117.2)
-		(width 0.5)
-		(layer "F.Cu")
-		(net 22)
-	)
-	(segment
-		(start 141.2 117.1)
-		(end 133.4 117.1)
-		(width 1)
-		(layer "F.Cu")
-		(net 22)
-	)
-	(segment
 		(start 141.8 88.2)
 		(end 143.61 88.2)
@@
 	)
 	(segment
-		(start 141.3 117.2)
-		(end 141.2 117.1)
-		(width 1)
-		(layer "F.Cu")
-		(net 22)
-	)
-	(segment
 		(start 140.9 89.1)
 		(end 141.8 88.2)
@@
 		(net 24)
 	)
+	(segment
+		(start 144.25 117.4)
+		(end 144.25 117.25)
+		(width 0.5)
+		(layer "F.Cu")
+		(net 25)
+	)
+	(segment
+		(start 144.25 117.25)
+		(end 144.2 117.2)
+		(width 0.5)
+		(layer "F.Cu")
+		(net 25)
+	)
+	(segment
+		(start 141.3 117.2)
+		(end 144.05 117.2)
+		(width 1)
+		(layer "F.Cu")
+		(net 25)
+	)
+	(segment
+		(start 141 116.9)
+		(end 141.3 117.2)
+		(width 1)
+		(layer "F.Cu")
+		(net 25)
+	)
+	(segment
+		(start 144.05 117.2)
+		(end 144.25 117.4)
+		(width 1)
+		(layer "F.Cu")
+		(net 25)
+	)
+	(segment
+		(start 133.4 116.9)
+		(end 141 116.9)
+		(width 1)
+		(layer "F.Cu")
+		(net 25)
+	)
 	(zone
